File: IM6100/front-panel.kicad_sch (KiCad schematic)
At the start: 99 parts, among them SW1 SS-12SDP2, SW10 SS-12SDP2, SW11 SS-12SDP2, SW12 SS-12SDP2, SW13 DTSM-644R-V-T/R, SW14 SS-12SDP2, SW15 DTSM-644R-V-T/R, SW16 DTSM-644R-V-T/R, SW17 SS-12SDP2, SW18 DTSM-644R-V-T/R, SW19 ERD216CSZ, SW2 SS-12SDP2, SW20 DTSM-644R-V-T/R, SW3 SS-12SDP2, SW4 SS-12SDP2, SW5 SS-12SDP2, SW6 SS-12SDP2, SW7 SS-12SDP2, SW8 SS-12SDP2, SW9 SS-12SDP2, U10 SN74LVC245APW, U11 SN74LVC574APW, U12 SN74LVC574APW, U7 SN74LVC574APW, U8 SN74LVC245APW, U9 SN74LVC574APW

Commit message: Updated tactile switch.
Parts:
- SW13, SW15, SW16, SW18, SW20: value DTSM-644R-V-T/R -> DTSM-63N-V-T/R; symbol 0my_project:DTSM-6x -> 0my_project:DTSM-63N-V-T/R; LCSC C483869 -> C133973
Changed lines of the file:
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@@
 	)
 	(symbol
-		(lib_id "0my_project:DTSM-6x")
+		(lib_id "0my_project:DTSM-63N-V-T/R")
 		(at 222.25 107.95 90)
 		(unit 1)
@@
 			)
 		)
-		(property "Value" "DTSM-644R-V-T/R"
-			(at 223.52 109.2199 90)
+		(property "Value" "DTSM-63N-V-T/R"
+			(at 224.79 107.95 0)
 			(effects
 				(font
 					(size 1.27 1.27)
 				)
-				(justify right)
 				(hide yes)
 			)
@@
 			)
 		)
-		(property "Datasheet" "https://datasheet.lcsc.com/lcsc/1811131733_Diptronics-DTSM-62R-V-T-R_C224979.pdf"
+		(property "Datasheet" "https://jlcpcb.com/api/file/downloadByFileSystemAccessId/8588899446814363648"
 			(at 222.25 107.95 0)
 			(effects
@@
 			)
 		)
-		(property "LCSC" "C483869"
+		(property "LCSC" "C133973"
 			(at 222.25 107.95 0)
 			(effects
@@
 	)
 	(symbol
-		(lib_id "0my_project:DTSM-6x")
+		(lib_id "0my_project:DTSM-63N-V-T/R")
 		(at 234.95 107.95 90)
 		(unit 1)
@@
 			)
 		)
-		(property "Value" "DTSM-644R-V-T/R"
-			(at 236.22 109.2199 90)
+		(property "Value" "DTSM-63N-V-T/R"
+			(at 237.49 107.95 0)
 			(effects
 				(font
 					(size 1.27 1.27)
 				)
-				(justify right)
 				(hide yes)
 			)
@@
 			)
 		)
-		(property "Datasheet" "https://datasheet.lcsc.com/lcsc/1811131733_Diptronics-DTSM-62R-V-T-R_C224979.pdf"
+		(property "Datasheet" "https://jlcpcb.com/api/file/downloadByFileSystemAccessId/8588899446814363648"
 			(at 234.95 107.95 0)
 			(effects
@@
 			)
 		)
-		(property "LCSC" "C483869"
+		(property "LCSC" "C133973"
 			(at 234.95 107.95 0)
 			(effects
@@
 	)
 	(symbol
-		(lib_id "0my_project:DTSM-6x")
+		(lib_id "0my_project:DTSM-63N-V-T/R")
 		(at 259.08 107.95 90)
 		(unit 1)
@@
 			)
 		)
-		(property "Value" "DTSM-644R-V-T/R"
-			(at 260.35 109.2199 90)
+		(property "Value" "DTSM-63N-V-T/R"
+			(at 261.62 107.95 0)
 			(effects
 				(font
 					(size 1.27 1.27)
 				)
-				(justify right)
 				(hide yes)
 			)
@@
 			)
 		)
-		(property "Datasheet" "https://datasheet.lcsc.com/lcsc/1811131733_Diptronics-DTSM-62R-V-T-R_C224979.pdf"
+		(property "Datasheet" "https://jlcpcb.com/api/file/downloadByFileSystemAccessId/8588899446814363648"
 			(at 259.08 107.95 0)
 			(effects
@@
 			)
 		)
-		(property "LCSC" "C483869"
+		(property "LCSC" "C133973"
 			(at 259.08 107.95 0)
 			(effects
@@
 	)
 	(symbol
-		(lib_id "0my_project:DTSM-6x")
+		(lib_id "0my_project:DTSM-63N-V-T/R")
 		(at 247.65 107.95 90)
 		(unit 1)
@@
 			)
 		)
-		(property "Value" "DTSM-644R-V-T/R"
-			(at 248.92 109.2199 90)
+		(property "Value" "DTSM-63N-V-T/R"
+			(at 250.19 107.95 0)
 			(effects
 				(font
 					(size 1.27 1.27)
 				)
-				(justify right)
 				(hide yes)
 			)
@@
 			)
 		)
-		(property "Datasheet" "https://datasheet.lcsc.com/lcsc/1811131733_Diptronics-DTSM-62R-V-T-R_C224979.pdf"
+		(property "Datasheet" "https://jlcpcb.com/api/file/downloadByFileSystemAccessId/8588899446814363648"
 			(at 247.65 107.95 0)
 			(effects
@@
 			)
 		)
-		(property "LCSC" "C483869"
+		(property "LCSC" "C133973"
 			(at 247.65 107.95 0)
 			(effects
@@
 	)
 	(symbol
-		(lib_id "0my_project:DTSM-6x")
+		(lib_id "0my_project:DTSM-63N-V-T/R")
 		(at 270.51 107.95 90)
 		(unit 1)
@@
 			)
 		)
-		(property "Value" "DTSM-644R-V-T/R"
-			(at 271.78 109.2199 90)
+		(property "Value" "DTSM-63N-V-T/R"
+			(at 273.05 107.95 0)
 			(effects
 				(font
 					(size 1.27 1.27)
 				)
-				(justify right)
 				(hide yes)
 			)
@@
 			)
 		)
-		(property "Datasheet" "https://datasheet.lcsc.com/lcsc/1811131733_Diptronics-DTSM-62R-V-T-R_C224979.pdf"
+		(property "Datasheet" "https://jlcpcb.com/api/file/downloadByFileSystemAccessId/8588899446814363648"
 			(at 270.51 107.95 0)
 			(effects
@@
 			)
 		)
-		(property "LCSC" "C483869"
+		(property "LCSC" "C133973"
 			(at 270.51 107.95 0)
 			(effects

Commit message: Replaced level shifter logics to SN74LVC8T245.
Parts:
- removed D27: OSR5JA5E34B, 0my_project:LED_5mm, symbol Device:LED
- removed R41: 1.2K, 0my_project:R_1608_0603, symbol Device:R
- removed R42: 10K, 0my_project:R_1608_0603, symbol Device:R
- removed SW13, SW15, SW16, SW18, SW20: DTSM-63N-V-T/R, 0my_project:DTSM-6x, symbol 0my_project:DTSM-63N-V-T/R
- removed SW14, SW17: SS-12SDP2, 0my_project:SS-12SDP2, symbol 0my_project:SS-12SDP2
- removed SW19: ERD216CSZ, 0my_project:ERD216CSZ, symbol 0my_project:ERD216CSZ
- added R19: 10K, 0my_project:R_1608_0603, symbol Device:R
- renumbered C12 to C14, C13 to C15, C14 to C16, C15 to C17, C16 to C18, C17 to C19, R11 to R10, R12 to R11, R13 to R12, R14 to R13, R15 to R14, R16 to R15, R17 to R16, R18 to R17, R19 to R18, R3 to R2, R23 to R21, R21 to R22, R22 to R23, R4 to R3, R5 to R4, R6 to R5, R7 to R6, R8 to R7, R9 to R8, R10 to R9, U7 to U11, U8 to U12, U9 to U13, U10 to U14, U11 to U15, U12 to U16
Connections:
- net +3.3V: now also R19.2
- net GND: now also U13.6 (D4), U13.7 (D5)
- net LINK_3V3: now also D14.2 (A); no longer U13.7 (D5)
- net RUN_3V3: now also D13.2 (A); no longer U13.6 (D4)
- net ~{SW_EN}: now also R19.1
- net at U13.14 (Q5): no longer D14.2 (A)
- net at U13.15 (Q4): no longer D13.2 (A)
- no-connect marks 25 -> 24
Other:
- note removed: "A single DMAGNT cycle is inserted at HALT to RUN transition. Single Step mode: RUN/HALT signal > wait aserting DMAGNT > wait deassertion > RUN/HALT signal."
- note removed: "Clear"
- note removed: "Control Panel Request"
- note removed: "DTSM-644R-V-T/R"
- note removed: "Dep"
- note removed: "Exam"
- note removed: "Internal Pull-up"
- note removed: "Load Addr"
- note removed: "Moniror items - Acc - MQ - Memory"
- note removed: "Monitor Select"
- note removed: "On: Autonomous CPREQ events"
- note removed: "Run/Halt"
- note removed: "Single Mode"
- note removed: "These SWs except RUN/HALT triger CPREQ."
- moved on the sheet: D13, D14, R22, R23
